File: PCB/iot_pwm_leddriver.kicad_pcb (KiCad board)
At the start: 4 copper layers, 55 x 35 mm, 53 parts, among them J1 ProgConn-SOICBite, J2 12V PWR, J3 LED_GRBWA, Q1 UMW30N06, Q2 UMW30N06, Q3 UMW30N06, Q4 UMW30N06, SW1 RESET, SW2 FLASH, U1 ESP-12F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

Commit message: schematic and layout cleanup
* plus BOM finalization
Parts:
- F2: footprint projectlib:FUSE-TH_XF-505P -> jmux-footprints:FUSE-TH_XF-505P
Routing:
- net /LED Driver/LED_B_GND: track 9.09 -> 8.18 mm
Changed lines of the file:
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@@
     (property "ki_keywords" "cap capacitor")
     (attr smd)
-    (fp_text reference "C5" (at -0.9625 -5.8) (layer "F.SilkS")
-        (effects (font (size 0.7 0.7) (thickness 0.11)))
+    (fp_text reference "C5" (at -0.0125 0.05) (layer "F.SilkS")
+        (effects (font (size 0.5 0.5) (thickness 0.09)))
     )
     (fp_text value "10uF" (at 0 1.68 90) (layer "F.Fab")
@@
     (tags "resistor handsolder")
     (property "LCSC" "C17414")
-    (property "Sheetfile" "dumb-led-driver.kicad_sch")
+    (property "Sheetfile" "iot_pwm_leddriver.kicad_sch")
     (property "Sheetname" "")
     (property "Vendor" "https://www.lcsc.com/product-detail/Chip-Resistor-Surface-Mount_FOJAN-FRQ0805F1002TS_C5159708.html")
@@
     (property "Description" "125mW Thick Film Resistors ±100ppm/℃ ±1% 1kΩ 0805 Chip Resistor - Surface Mount ROHS")
     (property "LCSC" " C17513 ")
-    (property "Sheetfile" "dumb-led-driver.kicad_sch")
+    (property "Sheetfile" "iot_pwm_leddriver.kicad_sch")
     (property "Sheetname" "")
     (property "Vendor" "")
@@
     (tags "resistor handsolder")
     (property "LCSC" "C17414")
-    (property "Sheetfile" "dumb-led-driver.kicad_sch")
+    (property "Sheetfile" "iot_pwm_leddriver.kicad_sch")
     (property "Sheetname" "")
     (property "Vendor" "https://www.lcsc.com/product-detail/Chip-Resistor-Surface-Mount_FOJAN-FRQ0805F1002TS_C5159708.html")
@@
     (tags "resistor handsolder")
     (property "LCSC" "C17414")
-    (property "Sheetfile" "dumb-led-driver.kicad_sch")
+    (property "Sheetfile" "iot_pwm_leddriver.kicad_sch")
     (property "Sheetname" "")
     (property "Vendor" "https://www.lcsc.com/product-detail/Chip-Resistor-Surface-Mount_FOJAN-FRQ0805F1002TS_C5159708.html")
@@
     (property "Description" "")
     (property "LCSC" "C15850")
-    (property "Sheetfile" "dumb-led-driver.kicad_sch")
+    (property "Sheetfile" "iot_pwm_leddriver.kicad_sch")
     (property "Sheetname" "")
     (property "Vendor" "https://www.lcsc.com/product-detail/Multilayer-Ceramic-Capacitors-MLCC-SMD-SMT_Murata-Electronics-GRM21BR61C106KE15L_C77075.html")
@@
     (tags "connector barrel jack")
     (property "LCSC" "C194407")
-    (property "Sheetfile" "dumb-led-driver.kicad_sch")
+    (property "Sheetfile" "iot_pwm_leddriver.kicad_sch")
     (property "Sheetname" "")
     (property "Vendor" "https://www.lcsc.com/product-detail/AC-span-style-background-color-ff0-DC-span-span-style-background-color-ff0-Power-span-Connectors_GANGYUAN-DC-470-2-1GP_C194407.html")
@@
     (tags "SPST Tactile Switch")
     (property "LCSC" "C318884")
-    (property "Sheetfile" "dumb-led-driver.kicad_sch")
+    (property "Sheetfile" "iot_pwm_leddriver.kicad_sch")
     (property "Sheetname" "")
     (property "Vendor" "https://www.lcsc.com/product-detail/Tactile-Switches_G-Switch-GT-TC060A-H025-L1_C5117870.html")
@@
     (descr "5-pin SOT23 package")
     (tags "SOT-23-5 hand-soldering")
+    (property "Description" "alternatively: https://www.lcsc.com/product-detail/Gate-Drive-ICs_JSMSEMI-MCP1416T-E-OT-JSM_C18195002.html")
     (property "LCSC" "C83775 ")
     (property "Sheetfile" "LED_driver.kicad_sch")
@@
     (descr "5-pin SOT23 package")
     (tags "SOT-23-5 hand-soldering")
+    (property "Description" "alternatively: https://www.lcsc.com/product-detail/Gate-Drive-ICs_JSMSEMI-MCP1416T-E-OT-JSM_C18195002.html")
     (property "LCSC" "C83775 ")
     (property "Sheetfile" "LED_driver.kicad_sch")
@@
     (descr "SOIC Bite Programming footprint: See https://github.com/SimonMerrett/SOICbite")
     (property "LCSC" "-")
-    (property "Sheetfile" "dumb-led-driver.kicad_sch")
+    (property "Sheetfile" "iot_pwm_leddriver.kicad_sch")
     (property "Sheetname" "")
     (property "exclude_from_bom" "")
@@
       (net 2 "Earth") (pinfunction "1") (pintype "input"))
   )
-  (footprint "projectlib:FUSE-TH_XF-505P" (layer "F.Cu")
+  (footprint "jmux-footprints:FUSE-TH_XF-505P" (layer "F.Cu")
     (at 127.75 71.9 90)
     (property "Description" "https://www.lcsc.com/product-detail/Fuse-Holders_XFCN-XF-505P_C843270.html")
@@
     (property "ki_keywords" "fuse")
     (attr through_hole)
-    (fp_text reference "F2" (at 0.15 0.15 90) (layer "F.SilkS")
+    (fp_text reference "F2" (at -0.05 0.35 90) (layer "F.SilkS")
         (effects (font (size 1 1) (thickness 0.15)))
     )
-    (fp_text value "Fuse Holder" (at -12.8 -4.55 180) (layer "F.Fab") hide
+    (fp_text value "Fuse Holder" (at 0 4 90) (layer "F.Fab")
         (effects (font (size 1 1) (thickness 0.15)))
     )
@@
     (pad "2" thru_hole oval (at 6 0 180) (size 2.3 1) (drill oval 1.900022 0.599999) (layers "*.Cu" "*.Mask")
       (net 3 "VDD") (pintype "passive"))
-    (model "/projectlib.3dshapes/FUSE-TH_XF-505P.wrl"
-      (offset (xyz -0.02 -0.62 0))
+    (model "${JMUX_KICAD_THINGS}/footprints/packages3d/FUSE-TH_XF-505P.wrl"
+      (offset (xyz 0 -0.5 0))
       (scale (xyz 1 1 1))
-      (rotate (xyz 0 0 180))
+      (rotate (xyz 0 0 -180))
     )
   )
@@
     (property "Description" "125mW Thick Film Resistors ±100ppm/℃ ±1% 1kΩ 0805 Chip Resistor - Surface Mount ROHS")
     (property "LCSC" " C17513 ")
-    (property "Sheetfile" "dumb-led-driver.kicad_sch")
+    (property "Sheetfile" "iot_pwm_leddriver.kicad_sch")
     (property "Sheetname" "")
     (property "Vendor" "")
@@
     (tags "resistor handsolder")
     (property "LCSC" "C17414")
-    (property "Sheetfile" "dumb-led-driver.kicad_sch")
+    (property "Sheetfile" "iot_pwm_leddriver.kicad_sch")
     (property "Sheetname" "")
     (property "Vendor" "https://www.lcsc.com/product-detail/Chip-Resistor-Surface-Mount_FOJAN-FRQ0805F1002TS_C5159708.html")
@@
     (property "ki_keywords" "cap capacitor")
     (attr smd)
-    (fp_text reference "C16" (at 0.8375 -1.8 unlocked) (layer "F.SilkS")
-        (effects (font (size 0.7 0.7) (thickness 0.11)))
+    (fp_text reference "C16" (at 0.0375 0 unlocked) (layer "F.SilkS")
+        (effects (font (size 0.5 0.5) (thickness 0.09)))
     )
     (fp_text value "100nF" (at 0 1.68 -90 unlocked) (layer "F.Fab") hide
@@
     (property "ki_keywords" "cap capacitor")
     (attr smd)
-    (fp_text reference "C17" (at -0.0625 -4 unlocked) (layer "F.SilkS")
-        (effects (font (size 0.7 0.7) (thickness 0.11)))
+    (fp_text reference "C17" (at -0.0125 0 unlocked) (layer "F.SilkS")
+        (effects (font (size 0.5 0.5) (thickness 0.09)))
     )
     (fp_text value "10uF" (at 0 1.68 -90 unlocked) (layer "F.Fab") hide
@@
     (tags "resistor handsolder")
     (property "LCSC" "C17414")
-    (property "Sheetfile" "dumb-led-driver.kicad_sch")
+    (property "Sheetfile" "iot_pwm_leddriver.kicad_sch")
     (property "Sheetname" "")
     (property "Vendor" "https://www.lcsc.com/product-detail/Chip-Resistor-Surface-Mount_FOJAN-FRQ0805F1002TS_C5159708.html")
@@
     (descr "5-pin SOT23 package")
     (tags "SOT-23-5 hand-soldering")
+    (property "Description" "alternatively: https://www.lcsc.com/product-detail/Gate-Drive-ICs_JSMSEMI-MCP1416T-E-OT-JSM_C18195002.html")
     (property "LCSC" "C83775 ")
     (property "Sheetfile" "LED_driver.kicad_sch")
@@
     (tags "LED handsolder")
     (property "LCSC" "C84256")
-    (property "Sheetfile" "dumb-led-driver.kicad_sch")
+    (property "Sheetfile" "iot_pwm_leddriver.kicad_sch")
     (property "Sheetname" "")
     (property "Vendor" "https://www.lcsc.com/product-detail/Light-Emitting-Diodes-LED_Foshan-NationStar-Optoelectronics-NCD1206B1_C130717.html")
@@
     (tags "SPST Tactile Switch")
     (property "LCSC" "C318884")
-    (property "Sheetfile" "dumb-led-driver.kicad_sch")
+    (property "Sheetfile" "iot_pwm_leddriver.kicad_sch")
     (property "Sheetname" "")
     (property "Vendor" "https://www.lcsc.com/product-detail/Tactile-Switches_G-Switch-GT-TC060A-H025-L1_C5117870.html")
@@
     (tags "LED handsolder")
     (property "LCSC" "C84256")
-    (property "Sheetfile" "dumb-led-driver.kicad_sch")
+    (property "Sheetfile" "iot_pwm_leddriver.kicad_sch")
     (property "Sheetname" "")
     (property "Vendor" "https://www.lcsc.com/product-detail/Light-Emitting-Diodes-LED_Foshan-NationStar-Optoelectronics-NCD1206B1_C130717.html")
@@
     (descr "5-pin SOT23 package")
     (tags "SOT-23-5 hand-soldering")
+    (property "Description" "alternatively: https://www.lcsc.com/product-detail/Gate-Drive-ICs_JSMSEMI-MCP1416T-E-OT-JSM_C18195002.html")
     (property "LCSC" "C83775 ")
     (property "Sheetfile" "LED_driver.kicad_sch")
@@
     (tags "Wi-Fi Module")
     (property "LCSC" " C82891 ")
-    (property "Sheetfile" "dumb-led-driver.kicad_sch")
+    (property "Sheetfile" "iot_pwm_leddriver.kicad_sch")
     (property "Sheetname" "")
     (property "ki_description" "802.11 b/g/n Wi-Fi Module")
@@
   (segment (start 137.952 60.35) (end 137.952 55.754) (width 2) (layer "B.Cu") (net 6))
   (segment (start 135.9 54.8) (end 136.998 54.8) (width 2) (layer "B.Cu") (net 6))
-  (segment (start 118.973 56.527) (end 118.973 54.977) (width 2) (layer "F.Cu") (net 7))
-  (segment (start 115.5 57.29) (end 118.21 57.29) (width 2) (layer "F.Cu") (net 7))
-  (segment (start 118.21 57.29) (end 118.973 56.527) (width 2) (layer "F.Cu") (net 7))
-  (segment (start 118.973 54.977) (end 121.625 52.325) (width 2) (layer "F.Cu") (net 7))
+  (segment (start 115.5 57.29) (end 116.66 57.29) (width 2) (layer "F.Cu") (net 7))
+  (segment (start 116.66 57.29) (end 121.625 52.325) (width 2) (layer "F.Cu") (net 7))
   (via (at 137.8 50.1) (size 1) (drill 0.7) (layers "F.Cu" "B.Cu") (free) (net 8))
   (via (at 137.8 51.3) (size 1) (drill 0.7) (layers "F.Cu" "B.Cu") (free) (net 8))
